Commit message: fix(ur5e): set gripper_tip offset to measured 211.4 mm
Calibrated tool0 -> gripper_tip_link to the measured value (FT300-S +
2F-85 stack). The 41.5 mm FT300-S envelope is unchanged, so the
gripper_tip joint origin moves from 0.163 to 0.1699 m relative to
robotiq_85_base_link.

The previous 0.163 m was a heritage value from o2ac-ur, flagged as
"not measured, needs calibration" by the xacro comment.

Header comment updated: FT300-S inertials are now overridden in
robotiq_ft300.urdf.xacro (loose third_party/robotiq repo), and the
2F-85 base mass is bumped in robotiq-cri's robotiq_arg2f.xacro to
match the catalog 0.925 kg.

Co-Authored-By: Claude <noreply@anthropic.com>

File: osx_ur5e/urdf/ur5e_ft300s_robotiq85.urdf.xacro (robot description, xacro)
@@ -4,10 +4,10 @@
      The FT300-S shares the FT300 mounting envelope (41.5 mm overall height,
      identical by Robotiq design), so the official ros-industrial robotiq_ft300
-     macro is reused for the kinematic chain. Inertial values in that macro are
-     the FT300 ones (mass 0.300 kg); the real FT300-S is 442 g with CoM
-     (-6, 0, 13.5) mm (manual section 5.2.1). They are left as-is here because
-     no consumer of this description uses the EE link inertials (robot_state_publisher
-     and the UR driver ignore them, and object inertial identification subtracts
-     the gripper contribution from real measurements after a zero calibration). -->
+     macro is reused for the kinematic chain. The macro's mass/CoM were
+     originally the FT300 values (300 g) — we now override them in
+     robotiq_ft300.urdf.xacro itself with the FT300-S figures (442 g, CoM
+     (-6, 0, 13.5) mm in the measurement frame, manual section 5.2.1).
+     Similarly, the 2F-85 base mass in robotiq_arg2f.xacro is bumped to make
+     the assembled gripper match the catalog 0.925 kg. -->
 <robot xmlns:xacro="http://www.ros.org/wiki/xacro" name="ur5e_ft300s_robotiq85">
   <!-- UR5e parameters -->
@@ -50,10 +50,10 @@
     <origin xyz="0 0 0.0415" rpy="0 ${-pi/2} ${pi/2}"/>
   </xacro:robotiq_85_gripper>
-  <!-- TCP: gripper tip link (163mm from robotiq_85_base_link along its X axis) -->
-  <!-- Matches the dual-arm setup in osx_end_effector.urdf.xacro -->
+  <!-- TCP: gripper tip link. 169.9 mm = measured tool0→tip (211.4 mm) minus
+       the 41.5 mm FT300-S stack above. -->
   <joint name="gripper_tip_joint" type="fixed">
     <parent link="robotiq_85_base_link"/>
     <child link="gripper_tip_link"/>
-    <origin xyz="0.163 0 0" rpy="0 0 0"/>
+    <origin xyz="0.1699 0 0" rpy="0 0 0"/>
   </joint>
   <link name="gripper_tip_link"/>

Commit message: feat(ur5e): unify URDF offsets and rename ft300s_sensor launch
- Set frame offsets for tool0-downward chain (FT300-S, coupling, gripper)
- Rename ft300_sensor.launch → ft300s_sensor.launch
- Rename robotiq_ft_frame_id → ft300s_measurement in launch default

Co-Authored-By: Claude <noreply@anthropic.com>

File: osx_ur5e/urdf/ur5e_ft300s_robotiq85.urdf.xacro (robot description, xacro)
@@ -25,5 +25,5 @@
   <xacro:include filename="$(find robotiq_description)/urdf/robotiq_85_gripper.urdf.xacro"/>
   <!-- Include official ros-industrial Robotiq FT300 macro (sensor + mounting plate) -->
-  <xacro:include filename="$(find robotiq_ft_sensor)/urdf/robotiq_ft300.urdf.xacro"/>
+  <xacro:include filename="$(find robotiq_ft_sensor)/urdf/robotiq_ft300s.urdf.xacro"/>
   <!-- Instantiate UR5e -->
   <xacro:ur5e_robot prefix=""
@@ -36,17 +36,36 @@
     safety_pos_margin="$(arg safety_pos_margin)"
     safety_k_position="$(arg safety_k_position)"/>
-  <!-- Attach Robotiq FT300-S (mounting plate + sensor) to the UR flange (tool0).
-       The official macro builds along +Z, and tool0 Z points forward, so an
-       identity origin mounts the plate flush on the flange. The assembly tool
-       face ends up at tool0 Z = 0.0415 m (13 mm plate + sensor body). -->
-  <xacro:robotiq_ft300 prefix="" parent="tool0">
-    <origin xyz="0 0 0" rpy="0 0 0"/>
-  </xacro:robotiq_ft300>
-  <!-- Attach Robotiq 2F-85 to the FT300-S tool face.
-       ft300_mounting_plate shares tool0's orientation, so place the gripper
-       0.0415 m forward (tool0 Z) and reuse the orientation that maps the
-       gripper X axis to the forward direction. -->
-  <xacro:robotiq_85_gripper prefix="" parent="ft300_mounting_plate">
-    <origin xyz="0 0 0.0415" rpy="0 ${-pi/2} ${pi/2}"/>
+  <!-- Attach Robotiq FT300-S to the UR flange (tool0) -->
+  <xacro:robotiq_ft300s prefix="" parent="tool0">
+    <origin xyz="0 0 0.0375" rpy="0 ${pi} 0"/>
+  </xacro:robotiq_ft300s>
+  <!-- Coupling plate between FT300-S and 2F-85.
+       ft300s_sensor frame is flipped (rpy=0,pi,0), so +Z in sensor frame
+       points toward tool0. Child offsets use negative Z to go forward. -->
+  <joint name="coupling_fix" type="fixed">
+    <origin xyz="0 0 0" rpy="0 ${-pi} 0"/>
+    <parent link="ft300s_sensor"/>
+    <child link="coupling_link"/>
+  </joint>
+  <link name="coupling_link">
+    <visual>
+      <origin xyz="0 0 0" rpy="0 0 0"/>
+      <geometry>
+        <mesh filename="package://robotiq_ft_sensor/meshes/visual/coupling_grp_es_cpl_062.stl" scale="0.001 0.001 0.001"/>
+      </geometry>
+      <material name="Robotiq-Grey">
+        <color rgba="0.4 0.4 0.4 1.0"/>
+      </material>
+    </visual>
+    <collision>
+      <origin xyz="0 0 0" rpy="0 0 0"/>
+      <geometry>
+        <mesh filename="package://robotiq_ft_sensor/meshes/collision/coupling_grp_es_cpl_062.stl" scale="0.001 0.001 0.001"/>
+      </geometry>
+    </collision>
+  </link>
+  <!-- Attach Robotiq 2F-85 to coupling plate -->
+  <xacro:robotiq_85_gripper prefix="" parent="coupling_link">
+    <origin xyz="0 0 0.011" rpy="0 ${-pi/2} ${pi/2}"/>
   </xacro:robotiq_85_gripper>
   <!-- TCP: gripper tip link. 169.9 mm = measured tool0→tip (211.4 mm) minus
